File: pigame_pico.kicad_pcb (KiCad board)
At the start: 2 copper layers, 139.7 x 64.8 mm, 41 parts, among them J1 1020_battery_holder, J2 Conn_PinHeader_2x03_P2.54mm_V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, SW1 W, SW2 A, SW3 S, SW4 D, SW5 I, SW6 J, SW7 K, SW8 L, SW9 Slideswitch, U1 Adafruit_TFT_ST7735, U2 MAX98357AETE+, U5 Pico

Commit message: update copper text
Parts:
- added Ref**: Val**, footprints:usb, B.Cu at (165.1, 63.5)
- moved G*** 3.65 mm to (117.0, 121.4)
- moved G*** 3.63 mm to (100.0, 121.4)
- moved G*** 1.34 mm to (202.0, 121.9)
